Commit message: Bake visual meshes into fr3.urdf, remove _inject_visual_meshes, clean up
- Modify fr3.urdf to include <visual> elements referencing STL meshes
- Remove _inject_visual_meshes from both franka.py and internal.py
- Inline mesh injection in franka.py robot_meta (for runtime URDF from C++ driver)
- Rename _REAL_ROBOT_META → REAL_ROBOT_META (public, used by eval.py)
- Inline _VIS_KEYS, remove # noqa hack

File: positronic/drivers/roboarm/fr3.urdf (robot description, URDF)
Before this commit: robot fr3, 11 links, 10 joints
Links:
- link link0: geometry visual mesh filename=link0.stl
- link link1: geometry visual mesh filename=link1.stl
- link link2: geometry visual mesh filename=link2.stl
- link link3: geometry visual mesh filename=link3.stl
- link link4: geometry visual mesh filename=link4.stl
- link link5: geometry visual mesh filename=link5.stl
- link link6: geometry visual mesh filename=link6.stl
- link link7: geometry visual mesh filename=link7.stl

Commit message: Fix URDF mesh paths in `_build_robot_meta` breaking 3D visualization
`_build_robot_meta` stored the libfranka URDF with `package://` mesh URIs
while the meshes dict used bare filenames. `_write_urdf_to_dir` couldn't
match them, Rerun failed to load the URDF, and all 3D pose entities got
"No transform path" errors.

Fix: rewrite all mesh refs to bare filenames matching the bundled STLs and
strip unresolvable .dae visuals. Regenerate `fr3.urdf` from the robot so
it matches `_build_robot_meta` output exactly.

File: positronic/drivers/roboarm/fr3.urdf (robot description, URDF)
Before this commit: robot fr3, 11 links, 10 joints
Links:
- link link0: geometry collision mesh filename=link0.stl; visual mesh filename=link0.stl
- link link1: geometry collision mesh filename=link1.stl; visual mesh filename=link1.stl
- link link2: geometry collision mesh filename=link2.stl; visual mesh filename=link2.stl
- link link3: geometry collision mesh filename=link3.stl; visual mesh filename=link3.stl
- link link4: geometry collision mesh filename=link4.stl; visual mesh filename=link4.stl
- link link5: geometry collision mesh filename=link5.stl; visual mesh filename=link5.stl
- link link6: geometry collision mesh filename=link6.stl; visual mesh filename=link6.stl
- link link7: geometry collision mesh filename=link7.stl; visual mesh filename=link7.stl
