Commit message: Use the sim panda joint limits in `panda.urdf`; inline `bundled_franka_model`
- Copy the panda joint ranges from `panda.xml` into `panda.urdf` — they differ from fr3's on every
  joint (joint6 most: -0.0175..3.7525 vs 0.5445..4.5169) — so `DLSIKSolverWithLimits` constrains sim
  IK solves to the real feasible set; assert the limits match `panda.xml` in the kinematics test
- Inline `bundled_franka_model()` in `_REAL_ROBOT_DERIVES` (it is lru-cached); drop `_FRANKA_MODEL`

File: positronic/assets/mujoco/panda.urdf (robot description, URDF)
Before this commit: robot panda, 12 links, 11 joints
Joints:
- joint joint1: limit lower=-2.7437 upper=2.7437 effort=87.0 velocity=2.62 -> lower=-2.8973 upper=2.8973 effort=87.0 velocity=2.62
- joint joint2: limit lower=-1.7837 upper=1.7837 effort=87.0 velocity=2.62 -> lower=-1.7628 upper=1.7628 effort=87.0 velocity=2.62
- joint joint3: limit lower=-2.9007 upper=2.9007 effort=87.0 velocity=2.62 -> lower=-2.8973 upper=2.8973 effort=87.0 velocity=2.62
- joint joint4: limit lower=-3.0421 upper=-0.1518 effort=87.0 velocity=2.62 -> lower=-3.0718 upper=-0.0698 effort=87.0 velocity=2.62
- joint joint5: limit lower=-2.8065 upper=2.8065 effort=12.0 velocity=5.26 -> lower=-2.8973 upper=2.8973 effort=12.0 velocity=5.26
- joint joint6: limit lower=0.5445 upper=4.5169 effort=12.0 velocity=4.18 -> lower=-0.0175 upper=3.7525 effort=12.0 velocity=4.18
- joint joint7: limit lower=-3.0159 upper=3.0159 effort=12.0 velocity=5.26 -> lower=-2.8973 upper=2.8973 effort=12.0 velocity=5.26

Commit message: Animate the sim gripper in the viewer from the `grip` signal
The panda finger joints were fixed, so the viewer showed a static gripper. Make `finger_joint1/2`
prismatic (0..0.04m, with the panda finger inertials so the moving bodies compile), add a `gripper`
spec to the emitted model (`signal=grip`, the two finger joints, travel), and have `_log_urdf_robot`
slide both fingers from the recorded [0,1] `grip`.

File: positronic/assets/mujoco/panda.urdf (robot description, URDF)
Before this commit: robot panda, 12 links, 11 joints
Links:
- link left_finger: mass None -> 0.015
- link right_finger: mass None -> 0.015
Joints:
- removed joint left_finger_joint
- removed joint right_finger_joint
- added joint finger_joint1: type prismatic, parent hand, child left_finger, origin xyz=0 0 0.0584 rpy=0 0 0, axis 0 1 0, limit lower=0 upper=0.04 effort=20 velocity=0.2
- added joint finger_joint2: type prismatic, parent hand, child right_finger, origin xyz=0 0 0.0584 rpy=0 0 3.141592653589793, axis 0 1 0, limit lower=0 upper=0.04 effort=20 velocity=0.2

Commit message: Mirror the sim gripper's right finger so the claws meet in the viewer

File: positronic/assets/mujoco/panda.urdf (robot description, URDF)
Before this commit: robot panda, 12 links, 11 joints
Joints:
- joint finger_joint2: axis 0 1 0 -> 0 -1 0
