Commit message: Unify gripper convention to 0 = open, 1 = closed
Flip the MuJoCo sim grip mapping, flip legacy sim recordings in the
dataset transforms, and serve inverted-grip checkpoints through a
`FlipGrip` codec.

File: positronic/assets/mujoco/panda.urdf (robot description, URDF)
Before this commit: robot panda, 12 links, 11 joints
Joints:
- joint finger_joint1: axis 0 1 0 -> 0 -1 0; origin xyz=0 0 0.0584 rpy=0 0 0 -> xyz=0 0.04 0.0584 rpy=0 0 0
- joint finger_joint2: axis 0 -1 0 -> 0 1 0; origin xyz=0 0 0.0584 rpy=0 0 3.141592653589793 -> xyz=0 -0.04 0.0584 rpy=0 0 3.141592653589793
