Commit message: Name the flange on the bundled sim panda
- Add `link8` to `panda.urdf`, 0.107 m along `link7` z with no rotation,
  and mount the hand on it, so the chain matches `fr3.urdf`.
- Add a `flange` site at the same place to `panda.xml`, `mjx_panda.xml`,
  `panda_ik.xml` and the `franka_table.xml` scene. The site is in group 4,
  so camera images do not change.
- `end_effector` and `default` stay where they are. No reported or solved
  pose changes.

The scene builder does not run on the locked MuJoCo, so `franka_table.xml`
gets the one site by hand.

Tests pin the flange on `link7`, the hand point 58.4 mm and -45deg off the
flange, and the MJCF flange sites against the recorded URDF at many joint
sets.

Ticket: Positronic-Robotics/internal#2298 #refs
Requested-by: Sergey Arkhangelskiy
Co-Authored-By: Claude Opus 5.5 (1M context) <noreply@anthropic.com>

File: positronic/assets/mujoco/panda.urdf (robot description, URDF)
Before this commit: robot panda, 12 links, 11 joints
Links:
- added link link8
Joints:
- added joint joint8: type fixed, parent link7, child link8, origin xyz=0 0 0.107 rpy=0 0 0
- joint hand_joint: origin xyz=0 0 0.107 rpy=0 0 -0.7853981633974483 -> xyz=0 0 0 rpy=0 0 -0.7853981633974483; parent link7 -> link8

Commit message: Name the grip point `gripper` on every bundled Franka model
- Rename the FR3 + 2F-85 site `gripper_grasp_site` to `gripper`, with one
  constant `GRIPPER_SITE` that `MolmoAdapter` and the tests read. It stays
  155 mm along the flange approach axis.
- Add a `gripper` link to `panda.urdf` under `link8`, 103.65 mm along the
  flange approach axis with no turn. Add the same site to `panda.xml`,
  `panda_ik.xml`, `mjx_panda.xml` and the `franka_table.xml` scene.
- `mjx_panda.xml` and `franka_table.xml` already had an unread `gripper`
  site on the hand, 100 mm out and turned -45deg. It moves to the new place
  and keeps its group, so the hand cameras still show it.
- No reported or solved pose changes: `default` stays where it is.

103.65 mm is the midpoint of the two fingertip pads of the sim scene. It is
the same at every arm pose and every finger opening, and a scene test pins it.

Ticket: Positronic-Robotics/internal#2298 #refs
Co-Authored-By: Claude Opus 5.5 (1M context) <noreply@anthropic.com>

File: positronic/assets/mujoco/panda.urdf (robot description, URDF)
Before this commit: robot panda, 13 links, 12 joints
Links:
- added link gripper
Joints:
- added joint gripper_joint: type fixed, parent link8, child gripper, origin xyz=0 0 0.10365 rpy=0 0 0
